Commit message: added mass and inertia properties

File: segway/urdf/segway.model.xacro (robot description, xacro)
@@ -19,4 +19,9 @@
     </geometry>
   </collision>
+  <inertial>
+    <origin rpy="0 0 0" xyz="0 0 0.5"/>
+    <mass value="5.0"/>
+    <inertia ixx="0.2" ixy="0.0" ixz="0.0" iyy="0.2" iyz="0.0" izz="0.1"/>
+  </inertial>
 </link>
 <!-- wheels for tracks -->

File: segway/urdf/segway_static.urdf (robot description, URDF)
Before this commit: robot segway, 3 links, 2 joints
Links:
- link base_frame: mass None -> 5.0

Commit message: now with wheel mass

File: segway/urdf/segway.model.xacro (robot description, xacro)
@@ -42,4 +42,9 @@
     </geometry>
   </collision>
+  <inertial>
+    <origin rpy="0 0 0" xyz="0 0 0"/>
+    <mass value="0.5"/>
+    <inertia ixx="0.001" ixy="0.0" ixz="0.0" iyy="0.001" iyz="0.0" izz="0.001"/>
+  </inertial>
 </link>
 <joint name="left_wheel_joint" type="continuous">
@@ -66,4 +71,9 @@
     </geometry>
   </collision>
+  <inertial>
+    <origin rpy="0 0 0" xyz="0 0 0"/>
+    <mass value="0.5"/>
+    <inertia ixx="0.001" ixy="0.0" ixz="0.0" iyy="0.001" iyz="0.0" izz="0.001"/>
+  </inertial>
 </link>
 <joint name="right_wheel_joint" type="continuous">

File: segway/urdf/segway_static.urdf (robot description, URDF)
Before this commit: robot segway, 3 links, 2 joints
Links:
- link left_wheel: mass None -> 0.5
- link right_wheel: mass None -> 0.5
